Commit message: auto push from scoot-motor

File: src/scootbot_description/src/description/scootbot_description.urdf (robot description, URDF)
Before this commit: robot scootbot, 2 links, 1 joints
Links:
- link base_link: geometry collision sphere radius=0.5 0.5; visual mesh filename=file:///home/teknetik/scootbot/install/scootbot_description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 scale=0.001 0.001 0.001
