Commit message: added tyre mesh

File: src/scootbot_description/src/description/gazebo_control.xacro (robot description, xacro)
@@ -4,6 +4,6 @@
         <plugin name="diff_drive" filename="libgazebo_ros_diff_drive.so">
         <!-- Wheel Information-->
-        <left_joint>drivewhl_l_link</left_joint>
-        <right_joint>drivewhl_r_link</right_joint>
+        <left_joint>drivewhl_l_joint</left_joint>
+        <right_joint>drivewhl_r_joint</right_joint>
         <wheel_seperation>0.44</wheel_seperation>
         <wheel_diameter>0.24</wheel_diameter>

File: src/scootbot_description/src/description/model.xacro (robot description, xacro)
@@ -8,9 +8,13 @@
 <!-- Measured from Fusion Model-->
   <xacro:property name="wheel_radius" value="0.12"/>
-  <xacro:property name="wheel_width" value="0.06"/>
-  <xacro:property name="wheel_ygap" value="0.245"/>
-  <xacro:property name="wheel_zoff" value="0.025"/>
+  <xacro:property name="wheel_width" value="0.05"/>
+  <xacro:property name="wheel_ygap" value="0.3"/>
+  <xacro:property name="wheel_zoff" value="0.01"/>
   <xacro:property name="wheel_xoff" value="0.20"/>
-  <xacro:property name="caster_xoff" value="0.14"/>
+  <xacro:property name="caster_radius" value="0.075"/>
+  <xacro:property name="caster_width" value="0.04"/>
+  <xacro:property name="caster_ygap" value="0.09"/>
+  <xacro:property name="caster_zoff" value="0.085"/>
+  <xacro:property name="caster_xoff" value="-0.26"/>
  <!-- Define intertial property macros  -->
   <xacro:macro name="box_inertia" params="m w h d">
@@ -37,6 +41,6 @@
   <link name="base_link">
     <visual>
-      <!-- <origin rpy="0 0 0" xyz="0.0 ${base_height/2} ${base_width/2}"/> -->
-      <origin rpy="0 0 0" xyz="0.0 -0.185 0.09"/>
+      <origin rpy="0 0 0" xyz="0.0 -0.18 0.10"/>
+      <!-- <origin rpy="0 0 0" xyz="0.0 0.0 0.0"/>  -->
       <geometry>
         <mesh filename="file:///home/teknetik/ros2_ws/install/scootbot_description/share/scootbot_description/src/description/frame.obj" scale="0.001 0.001 0.001"/>
@@ -47,10 +51,10 @@
     </visual>
    <collision>
-      <origin rpy="0 0 0" xyz="-1.0 0.0. 0.0"/>
+      <origin rpy="0 0 0" xyz="-1.0 0.0 0.0"/>
       <geometry>
-        <mesh filename="file:///home/teknetik/ros2_ws/install/scootbot_description/share/scootbot_description/src/description/frame.obj" scale="0.001 0.001 0.001"/>
+        <mesh filename="file:///home/ubuntu/scootbot/install/scootbot_description/share/scootbot_description/src/description/frame.obj" scale="0.001 0.001 0.001"/>
       </geometry>
     </collision>
-    <xacro:box_inertia m="15" w="${base_width}" d="${base_length}" h="${base_height}"/>
+    <xacro:box_inertia m="5" w="${base_width}" d="${base_length}" h="${base_height}"/>
   </link>
   <gazebo reference="base_link">
@@ -65,8 +69,11 @@
   </joint>
  <!-- Wheels -->
-  <xacro:macro name="wheel" params="prefix x_reflect y_reflect">
+  <xacro:macro name="wheel" params="prefix x_reflect y_reflect mirror x y">
     <link name="${prefix}_link">
       <visual>
-        <origin xyz="0 0 0" rpy="${pi/2} 0 0"/>
+        <origin xyz="${x} ${y} -0.135" rpy="${pi/2} 0 ${mirror} "/>
+        <geometry>
+        <mesh filename="file:///home/ubuntu/scootbot/install/scootbot_description/share/scootbot_description/src/description/tyre.obj" scale="0.002 0.002 0.002"/>
+      </geometry>
         <geometry>
             <cylinder radius="${wheel_radius}" length="${wheel_width}"/>
@@ -77,11 +84,23 @@
       </visual>
      <collision>
-        <origin xyz="0 0 0" rpy="${pi/2} 0 0"/>
+        <origin xyz="-0.135 -0.045 -0.135" rpy="${pi/2} 0 0"/>
         <geometry>
+        <mesh filename="file:///home/ubuntu/scootbot/install/scootbot_description/share/scootbot_description/src/description/tyre.obj" scale="0.002 0.002 0.002"/>
+      </geometry>
+        <!-- <geometry>
           <cylinder radius="${wheel_radius}" length="${wheel_width}"/>
-        </geometry>
+        </geometry> -->
       </collision>
       <xacro:cylinder_inertia m="0.5" r="${wheel_radius}" h="${wheel_width}"/>
     </link>
+    <gazebo reference="${prefix}_link">
+      <mu1 value="1.0"/>
+      <mu2 value="1.0"/>
+      <kp  value="10000000.0" />
+      <kd  value="1.0" />
+      <fdir1 value="1 0 0"/>
+      <material>Gazebo/Grey</material>
+    <turnGravityOff>false</turnGravityOff>
+</gazebo>
     <joint name="${prefix}_joint" type="continuous">
       <parent link="base_link"/>
@@ -91,21 +110,47 @@
     </joint>
   </xacro:macro>
-  <xacro:wheel prefix="drivewhl_l" x_reflect="1" y_reflect="0.43"/>
-  <xacro:wheel prefix="drivewhl_r" x_reflect="1" y_reflect="-0.47"/>
+  <xacro:wheel prefix="drivewhl_l" x_reflect="1" y_reflect="0.43" mirror="0" x="-0.135" y="-0.045"/>
+  <xacro:wheel prefix="drivewhl_r" x_reflect="1" y_reflect="-0.47" mirror="3.15" x="0.135" y="0.06"/>
  <!-- Caster Wheels -->
- <!-- <link name="front_caster">
-    <visual>
-      <geometry>
-        <sphere radius="${(wheel_radius+wheel_zoff-(base_height/2))}"/>
-      </geometry>
-      <material name="Cyan">
-        <color rgba="0 1.0 1.0 1.0"/>
-      </material>
-    </visual>
-  </link>
- <joint name="caster_joint" type="fixed">
-    <parent link="base_link"/>
-    <child link="front_caster"/>
-    <origin xyz="${caster_xoff} 0.0 ${-(base_height/2)}" rpy="0 0 0"/>
-  </joint>  -->
+  <xacro:macro name="caster_wheel" params="prefix x_reflect y_reflect">
+    <link name="${prefix}_link">
+      <visual>
+        <origin xyz="0 0 0" rpy="${pi/2} 0 0"/>
+        <geometry>
+            <cylinder radius="${caster_radius}" length="${caster_width}"/>
+        </geometry>
+        <material name="Gray">
+          <color rgba="0.5 0.5 0.5 1.0"/>
+        </material>
+      </visual>
+     <collision>
+        <origin xyz="0 0 0" rpy="${pi/2} 0 0"/>
+        <geometry>
+          <cylinder radius="${caster_radius}" length="${caster_width}"/>
+        </geometry>
+        <surface>
+        <friction>
+          <ode>
+            <mu>0.01</mu>
+            <mu2>0.01</mu2>
+          </ode>
+        </friction>
+        <contact>
+          <ode>
+            <min_depth>0.0</min_depth>
+          </ode>
+        </contact>
+      </surface>
+      </collision>
+      <xacro:cylinder_inertia m="0.5" r="${caster_radius}" h="${caster_width}"/>
+    </link>
+    <joint name="${prefix}_joint" type="continuous">
+      <parent link="base_link"/>
+      <child link="${prefix}_link"/>
+      <origin xyz="${x_reflect*caster_xoff} ${y_reflect*(base_width/2+caster_ygap)} ${-caster_zoff}" rpy="0 0 0"/>
+      <axis xyz="0 1 0"/>
+    </joint>
+  </xacro:macro>
+  <xacro:caster_wheel prefix="casterwhl_l" x_reflect="1" y_reflect="0.43"/>
+  <xacro:caster_wheel prefix="casterwhl_r" x_reflect="1" y_reflect="-0.47"/>
 </robot>

Commit message: README

File: src/scootbot_description/src/description/gazebo_control.xacro (robot description, xacro)
@@ -9,6 +9,6 @@
         <wheel_diameter>0.24</wheel_diameter>
         <!-- Limits -->
-        <max_wheel_torque>200</max_wheel_torque>
-        <max_wheel_acceleration>10</max_wheel_acceleration>
+        <max_wheel_torque>100</max_wheel_torque>
+        <max_wheel_acceleration>5</max_wheel_acceleration>
         <!-- Output-->
         <odometry_frame>odom</odometry_frame>

File: src/scootbot_description/src/description/model.xacro (robot description, xacro)
@@ -51,10 +51,14 @@
     </visual>
    <collision>
-      <origin rpy="0 0 0" xyz="-1.0 0.0 0.0"/>
+      <origin rpy="0 0 0" xyz="0.0 -0.18 0.10"/>
       <geometry>
         <mesh filename="file:///home/ubuntu/scootbot/install/scootbot_description/share/scootbot_description/src/description/frame.obj" scale="0.001 0.001 0.001"/>
       </geometry>
     </collision>
-    <xacro:box_inertia m="5" w="${base_width}" d="${base_length}" h="${base_height}"/>
+    <inertial>
+      <mass value="10.455"/>
+      <origin xyz="0.0 -0.18 0.10"/>
+      <inertia ixx="0.6022" ixy="-0.02364" ixz="-0.1197" iyy="1.7386" iyz="-0.001544" izz="2.0296"/>
+    </inertial>
   </link>
   <gazebo reference="base_link">
@@ -71,4 +75,15 @@
   <xacro:macro name="wheel" params="prefix x_reflect y_reflect mirror x y">
     <link name="${prefix}_link">
+    <contact>
+      <lateral_friction value="1.0"/>
+      <rolling_friction value="0.0"/>
+      <stiffness value="30000"/>
+      <damping value="1000"/>
+    </contact>
+    <inertial>
+      <mass value="2.637"/>
+      <origin xyz="0 0 0"/>
+      <inertia ixx="0.02467" ixy="0" ixz="0" iyy="0.02467" iyz="0" izz="0.04411"/>
+    </inertial>
       <visual>
         <origin xyz="${x} ${y} -0.135" rpy="${pi/2} 0 ${mirror} "/>
@@ -84,5 +99,5 @@
       </visual>
      <collision>
-        <origin xyz="-0.135 -0.045 -0.135" rpy="${pi/2} 0 0"/>
+        <origin xyz="${x} ${y} -0.135" rpy="${pi/2} 0 ${mirror} "/>
         <geometry>
         <mesh filename="file:///home/ubuntu/scootbot/install/scootbot_description/share/scootbot_description/src/description/tyre.obj" scale="0.002 0.002 0.002"/>
@@ -96,9 +111,9 @@
     <gazebo reference="${prefix}_link">
       <mu1 value="1.0"/>
-      <mu2 value="1.0"/>
-      <kp  value="10000000.0" />
-      <kd  value="1.0" />
-      <fdir1 value="1 0 0"/>
-      <material>Gazebo/Grey</material>
+    <mu2 value="1.0"/>
+    <kp value="10000000.0"/>
+    <kd value="1.0"/>
+    <fdir1 value="1 0 0"/>
+    <material>Gazebo/Grey</material>
     <turnGravityOff>false</turnGravityOff>
 </gazebo>
@@ -154,3 +169,25 @@
   <xacro:caster_wheel prefix="casterwhl_l" x_reflect="1" y_reflect="0.43"/>
   <xacro:caster_wheel prefix="casterwhl_r" x_reflect="1" y_reflect="-0.47"/>
+  <!-- BATTERY - Dimensions: (L) 181mm x (W) 76mm x (H) 167mm -->
+    <!-- <joint name="battery_joint" type="fixed">
+        <parent link="base_link"/>
+        <child link="battery"/>
+        <origin xyz="-0.1 0 0"/>
+    </joint>
+    <link name="battery">
+        <visual>
+            <origin xyz="0.06 0 0.03" rpy="0.0 0.0 0"/>
+            <geometry>
+                <box size="0.076 0.167 0.181"/>
+            </geometry>
+            <material name="white"/>
+        </visual>
+        <collision>
+            <origin xyz="0.06 0 0.03"/>
+            <geometry>
+                <box size="0.076 0.167 0.181"/>
+            </geometry>
+        </collision>
+        <xacro:box_inertia m="5" w="0.167" d="0.076" h="0.181"/>
+    </link> -->
 </robot>

Commit message: physics

File: src/scootbot_description/src/description/gazebo_control.xacro (robot description, xacro)
@@ -9,6 +9,6 @@
         <wheel_diameter>0.24</wheel_diameter>
         <!-- Limits -->
-        <max_wheel_torque>100</max_wheel_torque>
-        <max_wheel_acceleration>5</max_wheel_acceleration>
+        <max_wheel_torque>9</max_wheel_torque>
+        <max_wheel_acceleration>1</max_wheel_acceleration>
         <!-- Output-->
         <odometry_frame>odom</odometry_frame>

File: src/scootbot_description/src/description/model.xacro (robot description, xacro)
@@ -17,49 +17,37 @@
   <xacro:property name="caster_zoff" value="0.0985"/>
   <xacro:property name="caster_xoff" value="-0.0375"/>
- <!-- Define intertial property macros  -->
-  <xacro:macro name="box_inertia" params="m w h d">
-    <inertial>
-      <origin xyz="0 0 0" rpy="${pi/2} 0 ${pi/2}"/>
-      <mass value="${m}"/>
-      <inertia ixx="${(m/12) * (h*h + d*d)}" ixy="0.0" ixz="0.0" iyy="${(m/12) * (w*w + d*d)}" iyz="0.0" izz="${(m/12) * (w*w + h*h)}"/>
-    </inertial>
-  </xacro:macro>
-  <xacro:macro name="cylinder_inertia" params="m r h">
-    <inertial>
-      <origin xyz="0 0 0" rpy="${pi/2} 0 0" />
-      <mass value="${m}"/>
-      <inertia ixx="${(m/12) * (3*r*r + h*h)}" ixy = "0" ixz = "0" iyy="${(m/12) * (3*r*r + h*h)}" iyz = "0" izz="${(m/2) * (r*r)}"/>
-    </inertial>
-  </xacro:macro>
-  <xacro:macro name="sphere_inertia" params="m r">
-    <inertial>
-      <mass value="${m}"/>
-      <inertia ixx="${(2/5) * m * (r*r)}" ixy="0.0" ixz="0.0" iyy="${(2/5) * m * (r*r)}" iyz="0.0" izz="${(2/5) * m * (r*r)}"/>
-    </inertial>
-  </xacro:macro>
-  <!-- Robot Base -->
+<link name="dummy">
+   </link>
+<!-- Robot Base -->
   <link name="base_link">
     <visual>
       <origin rpy="0 0 0" xyz="0.0 -0.18 0.10"/>
-      <!-- <origin rpy="0 0 0" xyz="0.0 0.0 0.0"/>  -->
       <geometry>
-        <mesh filename="file:///home/ubuntu/scootbot/install/scootbot_description/share/scootbot_description/src/description/frame.obj" scale="0.001 0.001 0.001"/>
+        <mesh filename="file:///home/ubuntu/scootbot/install/scootbot_description/share/scootbot_description/src/description/frame.stl" scale="0.001 0.001 0.001"/>
       </geometry>
-       <material name="red">
-        <color rgba="1 0.4 0.4 1"/>
-      </material>
     </visual>
    <collision>
-      <origin rpy="0 0 0" xyz="0.0 -0.18 0.10"/>
+      <origin rpy="0 0 0" xyz="0 0 0.05 "/>
       <geometry>
-        <mesh filename="file:///home/ubuntu/scootbot/install/scootbot_description/share/scootbot_description/src/description/frame.obj" scale="0.001 0.001 0.001"/>
+        <!-- <mesh filename="file:///home/ubuntu/scootbot/install/scootbot_description/share/scootbot_description/src/description/frame.stl" scale="0.001 0.001 0.001"/> -->
+        <box size="0.663 0.39 0.312"/>
       </geometry>
     </collision>
     <inertial>
-      <mass value="10.455"/>
-      <origin xyz="0.0 -0.18 0.10"/>
-      <inertia ixx="0.6022" ixy="-0.02364" ixz="-0.1197" iyy="1.7386" iyz="-0.001544" izz="2.0296"/>
+      <mass value="10"/>
+      <origin xyz="0 0 0"/>
+      <!--
+        | ixx="-0.999998" ixy="-0.000077" ixz="0.001926" |
+        | ixy="-0.000078" iyy="1.000000" iyz="-0.000611" |
+        | ixz="-0.001926" iyz="-0.000611" izz="-0.999998" |
+        -->
+      <!-- <inertia ixx="-0.999998" ixy="-0.000077" ixz="-0.001926" iyy="1.000000" iyz="-0.000611" izz="-0.999998"/> -->
+      <inertia ixx="0" ixy="0" ixz="0" iyy="0" iyz="0" izz="0"/>
     </inertial>
   </link>
+  <joint name="dummy_joint" type="fixed">
+     <parent link="dummy"/>
+     <child link="base_link"/>
+   </joint>
   <gazebo reference="base_link">
     <material>Gazebo/Grey</material>
@@ -72,25 +60,27 @@
     <origin xyz="0.0 0.0 ${-(wheel_radius+wheel_zoff)}" rpy="0 0 0"/>
   </joint>
- <!-- Wheels -->
-  <xacro:macro name="wheel" params="prefix x_reflect y_reflect mirror x y">
-    <link name="${prefix}_link">
-    <contact>
+<!-- Wheels -->
+<xacro:macro name="wheel" params="prefix x_reflect y_reflect mirror x y col_x col_y col_z">
+  <link name="${prefix}_link">
+    <!-- <contact>
       <lateral_friction value="1.0"/>
       <rolling_friction value="0.0"/>
       <stiffness value="30000"/>
       <damping value="1000"/>
-    </contact>
+    </contact> -->
     <inertial>
-      <mass value="2.637"/>
+      <mass value="1"/>
       <origin xyz="0 0 0"/>
-      <inertia ixx="0.02467" ixy="0" ixz="0" iyy="0.02467" iyz="0" izz="0.04411"/>
+      <!--
+        | ixx="0.000819" ixy="-0.000000" ixz="0.000000" |
+        | ixy="-0.000000" iyy="0.001344" iyz="0.000000" |
+        | ixz="0.000000" iyz="0.000000" izz="0.000819" |
+        -->
+      <inertia ixx="0.000819" ixy="-0.000000" ixz="0.000000" iyy="0.001344" iyz="0.000000" izz="0.000819"/>
     </inertial>
       <visual>
         <origin xyz="${x} ${y} -0.135" rpy="${pi/2} 0 ${mirror} "/>
         <geometry>
-        <mesh filename="file:///home/ubuntu/scootbot/install/scootbot_description/share/scootbot_description/src/description/tyre.obj" scale="0.002 0.002 0.002"/>
-      </geometry>
-        <geometry>
-            <cylinder radius="${wheel_radius}" length="${wheel_width}"/>
+          <mesh filename="file:///home/ubuntu/scootbot/install/scootbot_description/share/scootbot_description/src/description/tyre.obj" scale="0.002 0.002 0.002"/>
         </geometry>
         <material name="Gray">
@@ -99,17 +89,16 @@
       </visual>
      <collision>
-        <origin xyz="${x} ${y} -0.135" rpy="${pi/2} 0 ${mirror} "/>
+        <origin xyz="${col_x} ${col_y} ${col_z}" rpy="${pi/2} 0 ${mirror} "/>
         <geometry>
-        <mesh filename="file:///home/ubuntu/scootbot/install/scootbot_description/share/scootbot_description/src/description/tyre.obj" scale="0.002 0.002 0.002"/>
-      </geometry>
-        <!-- <geometry>
-          <cylinder radius="${wheel_radius}" length="${wheel_width}"/>
-        </geometry> -->
+            <cylinder radius="0.135" length="0.09"/>
+        </geometry>
+        <material name="Gray">
+          <color rgba="0.5 0.5 0.5 1.0"/>
+        </material>
       </collision>
-      <xacro:cylinder_inertia m="0.5" r="${wheel_radius}" h="${wheel_width}"/>
     </link>
     <gazebo reference="${prefix}_link">
-      <mu1 value="1.0"/>
-      <mu2 value="1.0"/>
+      <mu1 value="100"/>
+      <mu2 value="100"/>
       <kp value="10000000.0"/>
       <kd value="1.0"/>
@@ -125,90 +114,5 @@
     </joint>
   </xacro:macro>
-  <xacro:wheel prefix="l" x_reflect="1" y_reflect="0.43" mirror="0" x="-0.135" y="-0.045"/>
-  <xacro:wheel prefix="r" x_reflect="1" y_reflect="-0.47" mirror="3.15" x="0.135" y="0.06"/>
- <!-- Caster Frame -->
-<xacro:macro name="caster_frame" params="prefix x_reflect y_reflect">
-    <link name="caster_frame_${prefix}_link">
-      <visual>
-        <origin xyz="0.22 -0.005 0.075" rpy="0 0 0"/>
-        <geometry>
-            <mesh filename="file:///home/ubuntu/scootbot/install/scootbot_description/share/scootbot_description/src/description/caster_frame.obj" scale="0.001 0.001 0.001"/>
-        </geometry>
-        <material name="Gray">
-          <color rgba="0.5 0.5 0.5 1.0"/>
-        </material>
-      </visual>
-     <collision>
-        <origin xyz="0 0 0" rpy="${pi/2} 0 0"/>
-        <geometry>
-          <cylinder radius="${caster_radius}" length="${caster_width}"/>
-        </geometry>
-      </collision>
-      <inertial>
-        <mass value="10.455"/>
-        <origin xyz="0.0 -0.18 0.10"/>
-        <inertia ixx="0.6022" ixy="-0.02364" ixz="-0.1197" iyy="1.7386" iyz="-0.001544" izz="2.0296"/>
-      </inertial>
-    </link>
-    <joint name="caster_frame_${prefix}_joint" type="continuous">
-      <parent link="base_link"/>
-      <child link="caster_frame_${prefix}_link"/>
-      <origin xyz="-0.221 ${y_reflect} 0.026" rpy="0 0 0"/>
-      <axis xyz="0 0 1"/>
-    </joint>
-    <gazebo reference="caster_frame_${prefix}_link">
-      <mu1 value="1.0"/>
-      <mu2 value="1.0"/>
-      <kp value="10000000.0"/>
-      <kd value="1.0"/>
-      <fdir1 value="1 0 0"/>
-      <material>Gazebo/Grey</material>
-      <turnGravityOff>false</turnGravityOff>
-    </gazebo>
-  </xacro:macro>
-<xacro:caster_frame prefix="l" x_reflect="1" y_reflect="-0.1752"/>
-<xacro:caster_frame prefix="r" x_reflect="1" y_reflect="0.1752"/>
- <!-- Caster Wheels -->
-  <xacro:macro name="caster_wheel" params="prefix x_reflect y_reflect">
-    <link name="casterwhl_${prefix}_link">
-      <visual>
-        <!-- <origin xyz="0.22 -0.165 -0.01" rpy="${pi/2} 0 0"/> -->
-        <origin xyz="0 0 0" rpy="${pi/2} 0 0"/>
-        <geometry>
-            <cylinder radius="${caster_radius}" length="${caster_width}"/>
-        </geometry>
-        <material name="Gray">
-          <color rgba="0.5 0.5 0.5 1.0"/>
-        </material>
-      </visual>
-     <collision>
-        <origin xyz="0 0 0" rpy="${pi/2} 0 0"/>
-        <geometry>
-          <cylinder radius="${caster_radius}" length="${caster_width}"/>
-        </geometry>
-        <surface>
-        <friction>
-          <ode>
-            <mu>0.01</mu>
-            <mu2>0.01</mu2>
-          </ode>
-        </friction>
-        <contact>
-          <ode>
-            <min_depth>0.0</min_depth>
-          </ode>
-        </contact>
-      </surface>
-      </collision>
-      <xacro:cylinder_inertia m="0.5" r="${caster_radius}" h="${caster_width}"/>
-    </link>
-    <joint name="casterwhl_${prefix}_joint" type="continuous">
-      <parent link="caster_frame_${prefix}_link"/>
-      <child link="casterwhl_${prefix}_link"/>
-      <origin xyz="${x_reflect*caster_xoff} ${y_reflect*(base_width/2+caster_ygap)} ${-caster_zoff}" rpy="0 0 0"/>
-      <axis xyz="0 1 0"/>
-    </joint>
-  </xacro:macro>
-  <xacro:caster_wheel prefix="l" x_reflect="1" y_reflect="0.43"/>
-  <xacro:caster_wheel prefix="r" x_reflect="1" y_reflect="-0.47"/>
+  <xacro:wheel prefix="l" x_reflect="1" y_reflect="0.43" mirror="0" x="-0.135" y="-0.05" col_x="0" col_y="0.0" col_z="0"/>
+  <xacro:wheel prefix="r" x_reflect="1" y_reflect="-0.47" mirror="3.15" x="0.135" y="0.065" col_x="0" col_y="0.015" col_z="0"/>
 </robot>
