Commit message: mapping and nav2

File: src/scootbot_description/src/description/gazebo_control.xacro (robot description, xacro)
@@ -6,8 +6,8 @@
         <left_joint>drivewhl_l_joint</left_joint>
         <right_joint>drivewhl_r_joint</right_joint>
-        <wheel_seperation>0.44</wheel_seperation>
+        <wheel_separation>0.44</wheel_separation>
         <wheel_diameter>0.24</wheel_diameter>
         <!-- Limits -->
-        <max_wheel_torque>9</max_wheel_torque>
+        <max_wheel_torque>10</max_wheel_torque>
         <max_wheel_acceleration>1</max_wheel_acceleration>
         <!-- Output-->

File: src/scootbot_description/src/description/model.xacro (robot description, xacro)
@@ -12,12 +12,18 @@
   <xacro:property name="wheel_zoff" value="0.01"/>
   <xacro:property name="wheel_xoff" value="0.20"/>
-  <xacro:property name="caster_radius" value="0.075"/>
+  <xacro:property name="caster_radius" value="0.071"/>
   <xacro:property name="caster_width" value="0.04"/>
   <xacro:property name="caster_ygap" value="-0.285"/>
   <xacro:property name="caster_zoff" value="0.0985"/>
   <xacro:property name="caster_xoff" value="-0.0375"/>
-<link name="dummy">
-   </link>
-<!-- Robot Base -->
+<!-- Robot base link -->
+  <link name="base_footprint">
+  </link>
+ <joint name="base_joint" type="fixed">
+    <parent link="base_link"/>
+    <child link="base_footprint"/>
+    <origin xyz="0.0 0.0 ${-(wheel_radius+wheel_zoff)}" rpy="0 0 0"/>
+  </joint>
+<!-- Robot Chassis -->
   <link name="base_link">
     <visual>
@@ -26,14 +32,17 @@
         <mesh filename="file:///home/ubuntu/scootbot/install/scootbot_description/share/scootbot_description/src/description/frame.stl" scale="0.001 0.001 0.001"/>
       </geometry>
+      <material name="Gray">
+          <color rgba="0.5 0.5 0.5 1.0"/>
+        </material>
     </visual>
    <collision>
-      <origin rpy="0 0 0" xyz="0 0 0.05 "/>
+      <origin rpy="0 0 0" xyz="0.05 0 -0.06 "/>
       <geometry>
         <!-- <mesh filename="file:///home/ubuntu/scootbot/install/scootbot_description/share/scootbot_description/src/description/frame.stl" scale="0.001 0.001 0.001"/> -->
-        <box size="0.663 0.39 0.312"/>
+        <box size="0.568 0.39 0.10"/>
       </geometry>
     </collision>
     <inertial>
-      <mass value="10"/>
+      <mass value="50"/>
       <origin xyz="0 0 0"/>
       <!--
@@ -46,29 +55,18 @@
     </inertial>
   </link>
-  <joint name="dummy_joint" type="fixed">
-     <parent link="dummy"/>
-     <child link="base_link"/>
-   </joint>
   <gazebo reference="base_link">
     <material>Gazebo/Grey</material>
   </gazebo>
-<!-- Robot Footprint -->
-  <link name="base_footprint"/>
- <joint name="base_joint" type="fixed">
-    <parent link="base_link"/>
-    <child link="base_footprint"/>
-    <origin xyz="0.0 0.0 ${-(wheel_radius+wheel_zoff)}" rpy="0 0 0"/>
-  </joint>
 <!-- Wheels -->
 <xacro:macro name="wheel" params="prefix x_reflect y_reflect mirror x y col_x col_y col_z">
   <link name="${prefix}_link">
-    <!-- <contact>
+    <contact>
       <lateral_friction value="1.0"/>
-      <rolling_friction value="0.0"/>
+      <rolling_friction value="1.0"/>
       <stiffness value="30000"/>
       <damping value="1000"/>
-    </contact> -->
+    </contact>
     <inertial>
-      <mass value="1"/>
+      <mass value="15"/>
       <origin xyz="0 0 0"/>
       <!--
@@ -91,5 +89,5 @@
         <origin xyz="${col_x} ${col_y} ${col_z}" rpy="${pi/2} 0 ${mirror} "/>
         <geometry>
-            <cylinder radius="0.135" length="0.09"/>
+            <cylinder radius="0.14" length="0.09"/>
         </geometry>
         <material name="Gray">
@@ -97,11 +95,11 @@
         </material>
       </collision>
-    </link>
+  </link>
     <gazebo reference="${prefix}_link">
-      <mu1 value="100"/>
-      <mu2 value="100"/>
+      <mu1 value="200"/>
+      <mu2 value="200"/>
       <kp value="10000000.0"/>
       <kd value="1.0"/>
-      <fdir1 value="1 0 0"/>
+      <minDepth>0.01</minDepth>
       <material>Gazebo/Grey</material>
       <turnGravityOff>false</turnGravityOff>
@@ -113,6 +111,153 @@
       <axis xyz="0 1 0"/>
     </joint>
+</xacro:macro>
+  <xacro:wheel prefix="l" x_reflect="1" y_reflect="0.43" mirror="0" x="-0.135" y="-0.05" col_x="0" col_y="0.0" col_z="0"/>
+  <xacro:wheel prefix="r" x_reflect="1" y_reflect="-0.47" mirror="3.15" x="0.135" y="0.065" col_x="0" col_y="0.0144" col_z="0"/>
+<!-- Caster Frame -->
+<xacro:macro name="caster_frame" params="prefix x_reflect y_reflect">
+    <link name="caster_frame_${prefix}_link">
+      <visual>
+        <origin xyz="0.22 -0.005 0.075" rpy="0 0 0"/>
+        <geometry>
+            <mesh filename="file:///home/ubuntu/scootbot/install/scootbot_description/share/scootbot_description/src/description/caster_frame.obj" scale="0.001 0.001 0.001"/>
+        </geometry>
+        <material name="Gray">
+          <color rgba="0.5 0.5 0.5 1.0"/>
+        </material>
+      </visual>
+     <collision>
+        <origin xyz="0.22 -0.005 0.075" rpy="0 0 0"/>
+        <geometry>
+          <mesh filename="file:///home/ubuntu/scootbot/install/scootbot_description/share/scootbot_description/src/description/caster_frame.obj" scale="0.001 0.001 0.001"/>
+        </geometry>
+      </collision>
+      <inertial>
+        <mass value="1"/>
+        <origin xyz="0 0 0" rpy="${pi/2} 0 0"/>
+        <inertia ixx="0.000419" ixy="-0.000000" ixz="0.000000" iyy="0.00744" iyz="0.000000" izz="0.000419"/>
+      </inertial>
+    </link>
+    <joint name="caster_frame_${prefix}_joint" type="continuous">
+      <parent link="base_link"/>
+      <child link="caster_frame_${prefix}_link"/>
+      <origin xyz="-0.221 ${y_reflect} 0.026" rpy="0 0 0"/>
+      <axis xyz="0 0 1"/>
+    </joint>
+    <gazebo reference="caster_frame_${prefix}_link">
+      <mu1 value="400"/>
+      <mu2 value="400"/>
+      <kp value="10000000.0"/>
+      <kd value="1.0"/>
+      <minDepth>0.01</minDepth>
+      <material>Gazebo/Grey</material>
+      <turnGravityOff>false</turnGravityOff>
+      <material>Gazebo/Grey</material>
+      <turnGravityOff>false</turnGravityOff>
+    </gazebo>
   </xacro:macro>
-  <xacro:wheel prefix="l" x_reflect="1" y_reflect="0.43" mirror="0" x="-0.135" y="-0.05" col_x="0" col_y="0.0" col_z="0"/>
-  <xacro:wheel prefix="r" x_reflect="1" y_reflect="-0.47" mirror="3.15" x="0.135" y="0.065" col_x="0" col_y="0.015" col_z="0"/>
+<xacro:caster_frame prefix="l" x_reflect="1" y_reflect="-0.1752"/>
+<xacro:caster_frame prefix="r" x_reflect="1" y_reflect="0.1752"/>
+ <!-- Caster Wheels -->
+  <xacro:macro name="caster_wheel" params="prefix x_reflect y_reflect">
+    <link name="casterwhl_${prefix}_link">
+      <visual>
+        <!-- <origin xyz="0.22 -0.165 -0.01" rpy="${pi/2} 0 0"/> -->
+        <origin xyz="0 0 0" rpy="${pi/2} 0 0"/>
+        <geometry>
+            <cylinder radius="${caster_radius}" length="${caster_width}"/>
+        </geometry>
+        <material name="Gray">
+          <color rgba="0.5 0.5 0.5 1.0"/>
+        </material>
+      </visual>
+     <collision>
+        <origin xyz="0 0 0" rpy="${pi/2} 0 0"/>
+        <geometry>
+          <cylinder radius="${caster_radius}" length="${caster_width}"/>
+        </geometry>
+      </collision>
+    <inertial>
+        <mass value="4"/>
+        <origin xyz="0 0 0" rpy="${pi/2} 0 0"/>
+        <inertia ixx="0.000419" ixy="-0.000000" ixz="0.000000" iyy="0.00744" iyz="0.000000" izz="0.000419"/>
+      </inertial>
+    </link>
+    <joint name="casterwhl_${prefix}_joint" type="continuous">
+      <parent link="caster_frame_${prefix}_link"/>
+      <child link="casterwhl_${prefix}_link"/>
+      <origin xyz="${x_reflect*caster_xoff} ${y_reflect*(base_width/2+caster_ygap)} ${-caster_zoff}" rpy="0 0 0"/>
+      <axis xyz="0 1 0"/>
+    </joint>
+    <gazebo reference="casterwhl_${prefix}_link">
+      <mu1 value="400"/>
+      <mu2 value="400"/>
+      <kp value="10000000.0"/>
+      <kd value="1.0"/>
+      <minDepth>0.01</minDepth>
+      <material>Gazebo/Grey</material>
+      <turnGravityOff>false</turnGravityOff>
+      <material>Gazebo/Grey</material>
+      <turnGravityOff>false</turnGravityOff>
+    </gazebo>
+  </xacro:macro>
+  <xacro:caster_wheel prefix="l" x_reflect="1" y_reflect="0.43"/>
+  <xacro:caster_wheel prefix="r" x_reflect="1" y_reflect="-0.47"/>
+ <joint name="laser_joint" type="fixed">
+        <parent link="base_link"/>
+        <child link="laser_frame"/>
+        <origin xyz="0.25 -0.005 0.18" rpy="0 0 0"/>
+    </joint>
+        <link name="laser_frame">
+      <visual>
+        <origin xyz="0 0 0" rpy="0 0 0"/>
+        <geometry>
+            <cylinder radius="0.04" length="0.04"/>
+        </geometry>
+      </visual>
+     <!-- <collision>
+        <origin xyz="0 0 0" rpy="0 0 0"/>
+        <geometry>
+          <cylinder radius="0.04" length="0.04"/>
+        </geometry>
+      </collision> -->
+    <!-- <inertial>
+        <mass value="1"/>
+        <origin xyz="0 0 0" rpy="0 0 0"/>
+        <inertia ixx="0.000419" ixy="-0.000000" ixz="0.000000" iyy="0.00744" iyz="0.000000" izz="0.000419"/>
+      </inertial> -->
+    </link>
+    <gazebo reference="laser_frame">
+        <mu1 value="400"/>
+        <mu2 value="400"/>
+        <kp value="10000000.0"/>
+        <kd value="1.0"/>
+        <minDepth>0.01</minDepth>
+        <material>Gazebo/Grey</material>
+        <turnGravityOff>false</turnGravityOff>
+        <sensor name="laser" type="ray">
+            <pose> 0 0 0 0 0.1 0 </pose>
+            <visualize>false</visualize>
+            <update_rate>10</update_rate>
+            <ray>
+                <scan>
+                    <horizontal>
+                        <samples>360</samples>
+                        <min_angle>-3.14</min_angle>
+                        <max_angle>3.14</max_angle>
+                    </horizontal>
+                </scan>
+                <range>
+                    <min>0.3</min>
+                    <max>12</max>
+                </range>
+            </ray>
+            <plugin name="laser_controller" filename="libgazebo_ros_ray_sensor.so">
+                <ros>
+                    <argument>~/out:=scan</argument>
+                </ros>
+                <output_type>sensor_msgs/LaserScan</output_type>
+                <frame_name>laser_frame</frame_name>
+            </plugin>
+        </sensor>
+    </gazebo>
 </robot>

Commit message: inertia

File: src/scootbot_description/src/description/gazebo_control.xacro (robot description, xacro)
@@ -9,6 +9,6 @@
         <wheel_diameter>0.24</wheel_diameter>
         <!-- Limits -->
-        <max_wheel_torque>10</max_wheel_torque>
-        <max_wheel_acceleration>1</max_wheel_acceleration>
+        <max_wheel_torque>5000</max_wheel_torque>
+        <max_wheel_acceleration>1.25</max_wheel_acceleration>
         <!-- Output-->
         <odometry_frame>odom</odometry_frame>

File: src/scootbot_description/src/description/model.xacro (robot description, xacro)
@@ -40,22 +40,24 @@
       <geometry>
         <!-- <mesh filename="file:///home/ubuntu/scootbot/install/scootbot_description/share/scootbot_description/src/description/frame.stl" scale="0.001 0.001 0.001"/> -->
-        <box size="0.568 0.39 0.10"/>
+        <box size="0.468 0.39 0.10"/>
       </geometry>
     </collision>
-    <inertial>
-      <mass value="50"/>
-      <origin xyz="0 0 0"/>
-      <!--
-        | ixx="-0.999998" ixy="-0.000077" ixz="0.001926" |
-        | ixy="-0.000078" iyy="1.000000" iyz="-0.000611" |
-        | ixz="-0.001926" iyz="-0.000611" izz="-0.999998" |
-        -->
-      <!-- <inertia ixx="-0.999998" ixy="-0.000077" ixz="-0.001926" iyy="1.000000" iyz="-0.000611" izz="-0.999998"/> -->
-      <inertia ixx="0" ixy="0" ixz="0" iyy="0" iyz="0" izz="0"/>
-    </inertial>
   </link>
   <gazebo reference="base_link">
     <material>Gazebo/Grey</material>
   </gazebo>
+ <!-- Inertial link stores the robot's inertial information -->
+  <link name="inertial_link">
+    <inertial>
+      <mass value="46.034" />
+      <origin xyz="0 0 0" />
+      <inertia ixx="0.6022" ixy="-0.02364" ixz="-0.1197" iyy="1.7386" iyz="-0.001544" izz="2.0296" />
+    </inertial>
+  </link>
+  <joint name="inertial_joint" type="fixed">
+    <origin xyz="0 0 0" rpy="0 0 0" />
+    <parent link="base_link" />
+    <child link="inertial_link" />
+  </joint>
 <!-- Wheels -->
 <xacro:macro name="wheel" params="prefix x_reflect y_reflect mirror x y col_x col_y col_z">
@@ -67,14 +69,9 @@
       <damping value="1000"/>
     </contact>
-    <inertial>
-      <mass value="15"/>
-      <origin xyz="0 0 0"/>
-      <!--
-        | ixx="0.000819" ixy="-0.000000" ixz="0.000000" |
-        | ixy="-0.000000" iyy="0.001344" iyz="0.000000" |
-        | ixz="0.000000" iyz="0.000000" izz="0.000819" |
-        -->
-      <inertia ixx="0.000819" ixy="-0.000000" ixz="0.000000" iyy="0.001344" iyz="0.000000" izz="0.000819"/>
-    </inertial>
+        <inertial>
+				<mass value="2.637" />
+				<origin xyz="0 0 0" />
+				<inertia  ixx="0.02467" ixy="0" ixz="0" iyy="0.04411" iyz="0" izz="0.02467" />
+			</inertial>
       <visual>
         <origin xyz="${x} ${y} -0.135" rpy="${pi/2} 0 ${mirror} "/>
@@ -97,12 +94,10 @@
   </link>
     <gazebo reference="${prefix}_link">
-      <mu1 value="200"/>
-      <mu2 value="200"/>
-      <kp value="10000000.0"/>
-      <kd value="1.0"/>
-      <minDepth>0.01</minDepth>
-      <material>Gazebo/Grey</material>
-      <turnGravityOff>false</turnGravityOff>
-    </gazebo>
+			<mu1 value="1.0"/>
+			<mu2 value="1.0"/>
+			<kp value="10000000.0" />
+			<kd value="1.0" />
+			<fdir1 value="1 0 0"/>
+		</gazebo>
     <joint name="drivewhl_${prefix}_joint" type="continuous">
       <parent link="base_link"/>
@@ -133,8 +128,8 @@
       </collision>
       <inertial>
-        <mass value="1"/>
-        <origin xyz="0 0 0" rpy="${pi/2} 0 0"/>
-        <inertia ixx="0.000419" ixy="-0.000000" ixz="0.000000" iyy="0.00744" iyz="0.000000" izz="0.000419"/>
-      </inertial>
+				<mass value="2.637" />
+				<origin xyz="0 0 0" />
+				<inertia  ixx="0.0002467" ixy="0" ixz="0" iyy="0.0004411" iyz="0" izz="0.0002467" />
+			</inertial>
     </link>
     <joint name="caster_frame_${prefix}_joint" type="continuous">
@@ -145,13 +140,9 @@
     </joint>
     <gazebo reference="caster_frame_${prefix}_link">
-      <mu1 value="400"/>
-      <mu2 value="400"/>
-      <kp value="10000000.0"/>
-      <kd value="1.0"/>
-      <minDepth>0.01</minDepth>
-      <material>Gazebo/Grey</material>
-      <turnGravityOff>false</turnGravityOff>
-      <material>Gazebo/Grey</material>
-      <turnGravityOff>false</turnGravityOff>
+      <mu1 value="1.0"/>
+			<mu2 value="1.0"/>
+			<kp value="10000000.0" />
+			<kd value="1.0" />
+			<fdir1 value="1 0 0"/>
     </gazebo>
   </xacro:macro>
@@ -174,12 +165,13 @@
         <origin xyz="0 0 0" rpy="${pi/2} 0 0"/>
         <geometry>
-          <cylinder radius="${caster_radius}" length="${caster_width}"/>
+          <!-- <cylinder radius="${caster_radius}" length="${caster_width}"/> -->
+          <sphere radius="${caster_radius}"/>
         </geometry>
       </collision>
-    <inertial>
-        <mass value="4"/>
-        <origin xyz="0 0 0" rpy="${pi/2} 0 0"/>
-        <inertia ixx="0.000419" ixy="-0.000000" ixz="0.000000" iyy="0.00744" iyz="0.000000" izz="0.000419"/>
-      </inertial>
+          <inertial>
+				<mass value="2.637" />
+				<origin xyz="0 0 0" />
+				<inertia  ixx="0.0002467" ixy="0" ixz="0" iyy="0.0004411" iyz="0" izz="0.0002467" />
+			</inertial>
     </link>
     <joint name="casterwhl_${prefix}_joint" type="continuous">
@@ -190,13 +182,9 @@
     </joint>
     <gazebo reference="casterwhl_${prefix}_link">
-      <mu1 value="400"/>
-      <mu2 value="400"/>
-      <kp value="10000000.0"/>
-      <kd value="1.0"/>
-      <minDepth>0.01</minDepth>
-      <material>Gazebo/Grey</material>
-      <turnGravityOff>false</turnGravityOff>
-      <material>Gazebo/Grey</material>
-      <turnGravityOff>false</turnGravityOff>
+      <mu1 value="1.0"/>
+			<mu2 value="1.0"/>
+			<kp value="10000000.0" />
+			<kd value="1.0" />
+			<fdir1 value="1 0 0"/>
     </gazebo>
   </xacro:macro>
