Commit message: gazebo

File: src/scootbot_description/src/description/model.xacro (robot description, xacro)
@@ -40,5 +40,5 @@
       <origin rpy="0 0 0" xyz="0.0 -0.185 0.09"/>
       <geometry>
-        <mesh filename="file:///home/teknetik/scootbot/install/scootbot_description/share/scootbot_description/src/description/frame.obj" scale="0.001 0.001 0.001"/>
+        <mesh filename="file:///home/teknetik/ros2_ws/install/scootbot_description/share/scootbot_description/src/description/frame.obj" scale="0.001 0.001 0.001"/>
       </geometry>
        <material name="red">
@@ -47,10 +47,14 @@
     </visual>
    <collision>
+      <origin rpy="0 0 0" xyz="-1.0 0.0. 0.0"/>
       <geometry>
-        <sphere radius="0.5 0.5"/>
+        <mesh filename="file:///home/teknetik/ros2_ws/install/scootbot_description/share/scootbot_description/src/description/frame.obj" scale="0.001 0.001 0.001"/>
       </geometry>
     </collision>
     <xacro:box_inertia m="15" w="${base_width}" d="${base_length}" h="${base_height}"/>
   </link>
+  <gazebo reference="base_link">
+    <material>Gazebo/Grey</material>
+  </gazebo>
 <!-- Robot Footprint -->
   <link name="base_footprint"/>

File: src/scootbot_description/src/description/scootbot_description.urdf (robot description, URDF)
Before this commit: robot scootbot, 2 links, 1 joints
Links:
- removed link base_footprint
- removed link base_link
Joints:
- removed joint base_joint

Commit message: add castors

File: src/scootbot_description/src/description/model.xacro (robot description, xacro)
@@ -14,7 +14,7 @@
   <xacro:property name="caster_radius" value="0.075"/>
   <xacro:property name="caster_width" value="0.04"/>
-  <xacro:property name="caster_ygap" value="0.09"/>
-  <xacro:property name="caster_zoff" value="0.085"/>
-  <xacro:property name="caster_xoff" value="-0.26"/>
+  <xacro:property name="caster_ygap" value="-0.285"/>
+  <xacro:property name="caster_zoff" value="0.0985"/>
+  <xacro:property name="caster_xoff" value="-0.0375"/>
  <!-- Define intertial property macros  -->
   <xacro:macro name="box_inertia" params="m w h d">
@@ -44,5 +44,5 @@
       <!-- <origin rpy="0 0 0" xyz="0.0 0.0 0.0"/>  -->
       <geometry>
-        <mesh filename="file:///home/teknetik/ros2_ws/install/scootbot_description/share/scootbot_description/src/description/frame.obj" scale="0.001 0.001 0.001"/>
+        <mesh filename="file:///home/ubuntu/scootbot/install/scootbot_description/share/scootbot_description/src/description/frame.obj" scale="0.001 0.001 0.001"/>
       </geometry>
        <material name="red">
@@ -118,5 +118,5 @@
     <turnGravityOff>false</turnGravityOff>
 </gazebo>
-    <joint name="${prefix}_joint" type="continuous">
+    <joint name="drivewhl_${prefix}_joint" type="continuous">
       <parent link="base_link"/>
       <child link="${prefix}_link"/>
@@ -125,10 +125,38 @@
     </joint>
   </xacro:macro>
-  <xacro:wheel prefix="drivewhl_l" x_reflect="1" y_reflect="0.43" mirror="0" x="-0.135" y="-0.045"/>
-  <xacro:wheel prefix="drivewhl_r" x_reflect="1" y_reflect="-0.47" mirror="3.15" x="0.135" y="0.06"/>
+  <xacro:wheel prefix="l" x_reflect="1" y_reflect="0.43" mirror="0" x="-0.135" y="-0.045"/>
+  <xacro:wheel prefix="r" x_reflect="1" y_reflect="-0.47" mirror="3.15" x="0.135" y="0.06"/>
+ <!-- Caster Frame -->
+<xacro:macro name="caster_frame" params="prefix x_reflect y_reflect">
+    <link name="caster_frame_${prefix}_link">
+      <visual>
+        <origin xyz="0.22 -0.005 0.075" rpy="0 0 0"/>
+        <geometry>
+            <mesh filename="file:///home/ubuntu/scootbot/install/scootbot_description/share/scootbot_description/src/description/caster_frame.obj" scale="0.001 0.001 0.001"/>
+        </geometry>
+        <material name="Gray">
+          <color rgba="0.5 0.5 0.5 1.0"/>
+        </material>
+      </visual>
+     <collision>
+        <origin xyz="0 0 0" rpy="${pi/2} 0 0"/>
+        <geometry>
+          <cylinder radius="${caster_radius}" length="${caster_width}"/>
+        </geometry>
+      </collision>
+    </link>
+    <joint name="caster_frame_${prefix}_joint" type="continuous">
+      <parent link="base_link"/>
+      <child link="caster_frame_${prefix}_link"/>
+      <origin xyz="-0.221 -0.1752 0.026" rpy="0 0 0"/>
+      <axis xyz="0 0 1"/>
+    </joint>
+  </xacro:macro>
+<xacro:caster_frame prefix="l" x_reflect="1" y_reflect="0.43"/>
  <!-- Caster Wheels -->
   <xacro:macro name="caster_wheel" params="prefix x_reflect y_reflect">
-    <link name="${prefix}_link">
+    <link name="casterwhl_${prefix}_link">
       <visual>
+        <!-- <origin xyz="0.22 -0.165 -0.01" rpy="${pi/2} 0 0"/> -->
         <origin xyz="0 0 0" rpy="${pi/2} 0 0"/>
         <geometry>
@@ -160,34 +188,12 @@
       <xacro:cylinder_inertia m="0.5" r="${caster_radius}" h="${caster_width}"/>
     </link>
-    <joint name="${prefix}_joint" type="continuous">
-      <parent link="base_link"/>
-      <child link="${prefix}_link"/>
+    <joint name="casterwhl_${prefix}_joint" type="continuous">
+      <parent link="caster_frame_${prefix}_link"/>
+      <child link="casterwhl_${prefix}_link"/>
       <origin xyz="${x_reflect*caster_xoff} ${y_reflect*(base_width/2+caster_ygap)} ${-caster_zoff}" rpy="0 0 0"/>
       <axis xyz="0 1 0"/>
     </joint>
   </xacro:macro>
-  <xacro:caster_wheel prefix="casterwhl_l" x_reflect="1" y_reflect="0.43"/>
-  <xacro:caster_wheel prefix="casterwhl_r" x_reflect="1" y_reflect="-0.47"/>
-  <!-- BATTERY - Dimensions: (L) 181mm x (W) 76mm x (H) 167mm -->
-    <!-- <joint name="battery_joint" type="fixed">
-        <parent link="base_link"/>
-        <child link="battery"/>
-        <origin xyz="-0.1 0 0"/>
-    </joint>
-    <link name="battery">
-        <visual>
-            <origin xyz="0.06 0 0.03" rpy="0.0 0.0 0"/>
-            <geometry>
-                <box size="0.076 0.167 0.181"/>
-            </geometry>
-            <material name="white"/>
-        </visual>
-        <collision>
-            <origin xyz="0.06 0 0.03"/>
-            <geometry>
-                <box size="0.076 0.167 0.181"/>
-            </geometry>
-        </collision>
-        <xacro:box_inertia m="5" w="0.167" d="0.076" h="0.181"/>
-    </link> -->
+  <xacro:caster_wheel prefix="l" x_reflect="1" y_reflect="0.43"/>
+  <!-- <xacro:caster_wheel prefix="r" x_reflect="1" y_reflect="-0.47"/> -->
 </robot>

Commit message: wheels!!

File: src/scootbot_description/src/description/model.xacro (robot description, xacro)
@@ -111,11 +111,11 @@
     <gazebo reference="${prefix}_link">
       <mu1 value="1.0"/>
-    <mu2 value="1.0"/>
-    <kp value="10000000.0"/>
-    <kd value="1.0"/>
-    <fdir1 value="1 0 0"/>
-    <material>Gazebo/Grey</material>
-    <turnGravityOff>false</turnGravityOff>
-</gazebo>
+      <mu2 value="1.0"/>
+      <kp value="10000000.0"/>
+      <kd value="1.0"/>
+      <fdir1 value="1 0 0"/>
+      <material>Gazebo/Grey</material>
+      <turnGravityOff>false</turnGravityOff>
+    </gazebo>
     <joint name="drivewhl_${prefix}_joint" type="continuous">
       <parent link="base_link"/>
@@ -145,13 +145,28 @@
         </geometry>
       </collision>
+      <inertial>
+        <mass value="10.455"/>
+        <origin xyz="0.0 -0.18 0.10"/>
+        <inertia ixx="0.6022" ixy="-0.02364" ixz="-0.1197" iyy="1.7386" iyz="-0.001544" izz="2.0296"/>
+      </inertial>
     </link>
     <joint name="caster_frame_${prefix}_joint" type="continuous">
       <parent link="base_link"/>
       <child link="caster_frame_${prefix}_link"/>
-      <origin xyz="-0.221 -0.1752 0.026" rpy="0 0 0"/>
+      <origin xyz="-0.221 ${y_reflect} 0.026" rpy="0 0 0"/>
       <axis xyz="0 0 1"/>
     </joint>
-  </xacro:macro>
-<xacro:caster_frame prefix="l" x_reflect="1" y_reflect="0.43"/>
+    <gazebo reference="caster_frame_${prefix}_link">
+      <mu1 value="1.0"/>
+      <mu2 value="1.0"/>
+      <kp value="10000000.0"/>
+      <kd value="1.0"/>
+      <fdir1 value="1 0 0"/>
+      <material>Gazebo/Grey</material>
+      <turnGravityOff>false</turnGravityOff>
+    </gazebo>
+  </xacro:macro>
+<xacro:caster_frame prefix="l" x_reflect="1" y_reflect="-0.1752"/>
+<xacro:caster_frame prefix="r" x_reflect="1" y_reflect="0.1752"/>
  <!-- Caster Wheels -->
   <xacro:macro name="caster_wheel" params="prefix x_reflect y_reflect">
@@ -196,4 +211,4 @@
   </xacro:macro>
   <xacro:caster_wheel prefix="l" x_reflect="1" y_reflect="0.43"/>
-  <!-- <xacro:caster_wheel prefix="r" x_reflect="1" y_reflect="-0.47"/> -->
+  <xacro:caster_wheel prefix="r" x_reflect="1" y_reflect="-0.47"/>
 </robot>

Commit message: more inertial fixes

File: src/scootbot_description/src/description/model.xacro (robot description, xacro)
@@ -1,4 +1,5 @@
 <?xml version="1.0"?>
 <robot xmlns:xacro="http://ros.org/wiki/xacro">
+<xacro:include filename="inertial_macros.xacro"/>
 <!-- Define robot constants -->
 <!-- Measured from Fusion Model-->
@@ -13,5 +14,5 @@
   <xacro:property name="wheel_xoff" value="0.20"/>
   <xacro:property name="caster_radius" value="0.071"/>
-  <xacro:property name="caster_width" value="0.04"/>
+  <xacro:property name="caster_width" value="0.047"/>
   <xacro:property name="caster_ygap" value="-0.285"/>
   <xacro:property name="caster_zoff" value="0.0985"/>
@@ -47,14 +48,17 @@
     <material>Gazebo/Grey</material>
   </gazebo>
- <!-- Inertial link stores the robot's inertial information -->
+ <!-- Inertial link stores the robot's inertial information - Chassis (31 Kg) + 2x Battery (5.5 Kg Each) = 42 Kg -->
   <link name="inertial_link">
-    <inertial>
+    <xacro:inertial_box mass="42" x="0.5" y="0.4" z="0.21">
+            <origin xyz="0.1 0 0" rpy="0 0 0"/>
+    </xacro:inertial_box>
+    <!-- <inertial>
       <mass value="46.034" />
       <origin xyz="0 0 0" />
       <inertia ixx="0.6022" ixy="-0.02364" ixz="-0.1197" iyy="1.7386" iyz="-0.001544" izz="2.0296" />
-    </inertial>
+    </inertial> -->
   </link>
   <joint name="inertial_joint" type="fixed">
-    <origin xyz="0 0 0" rpy="0 0 0" />
+    <origin xyz="0 0 0.02" rpy="0 0 0" />
     <parent link="base_link" />
     <child link="inertial_link" />
@@ -69,9 +73,7 @@
       <damping value="1000"/>
     </contact>
-        <inertial>
-				<mass value="2.637" />
-				<origin xyz="0 0 0" />
-				<inertia  ixx="0.02467" ixy="0" ixz="0" iyy="0.04411" iyz="0" izz="0.02467" />
-			</inertial>
+    <xacro:inertial_cylinder mass="2" length="0.08" radius="0.125">
+      <origin xyz="0 0 0" rpy="0 0 0"/>
+    </xacro:inertial_cylinder>
       <visual>
         <origin xyz="${x} ${y} -0.135" rpy="${pi/2} 0 ${mirror} "/>
@@ -127,9 +129,7 @@
         </geometry>
       </collision>
-      <inertial>
-				<mass value="2.637" />
-				<origin xyz="0 0 0" />
-				<inertia  ixx="0.0002467" ixy="0" ixz="0" iyy="0.0004411" iyz="0" izz="0.0002467" />
-			</inertial>
+      <xacro:inertial_box mass="1.5" x="0.05" y="0.1" z="0.1">
+        <origin xyz="0 0 0" rpy="0 0 0"/>
+      </xacro:inertial_box>
     </link>
     <joint name="caster_frame_${prefix}_joint" type="continuous">
@@ -149,5 +149,5 @@
 <xacro:caster_frame prefix="l" x_reflect="1" y_reflect="-0.1752"/>
 <xacro:caster_frame prefix="r" x_reflect="1" y_reflect="0.1752"/>
- <!-- Caster Wheels -->
+<!-- Caster Wheels -->
   <xacro:macro name="caster_wheel" params="prefix x_reflect y_reflect">
     <link name="casterwhl_${prefix}_link">
@@ -165,13 +165,11 @@
         <origin xyz="0 0 0" rpy="${pi/2} 0 0"/>
         <geometry>
-          <!-- <cylinder radius="${caster_radius}" length="${caster_width}"/> -->
-          <sphere radius="${caster_radius}"/>
+          <cylinder radius="0.075" length="0.05"/>
+          <!-- <sphere radius="0.1"/> -->
         </geometry>
       </collision>
-          <inertial>
-				<mass value="2.637" />
-				<origin xyz="0 0 0" />
-				<inertia  ixx="0.0002467" ixy="0" ixz="0" iyy="0.0004411" iyz="0" izz="0.0002467" />
-			</inertial>
+      <xacro:inertial_cylinder mass="0.586" length="${caster_width}" radius="${caster_radius}">
+        <origin xyz="0 0 0" rpy="0 0 0"/>
+      </xacro:inertial_cylinder>
     </link>
     <joint name="casterwhl_${prefix}_joint" type="continuous">
@@ -189,5 +187,5 @@
     </gazebo>
   </xacro:macro>
-  <xacro:caster_wheel prefix="l" x_reflect="1" y_reflect="0.43"/>
+  <xacro:caster_wheel prefix="l" x_reflect="1" y_reflect="0.47"/>
   <xacro:caster_wheel prefix="r" x_reflect="1" y_reflect="-0.47"/>
  <joint name="laser_joint" type="fixed">
@@ -215,5 +213,5 @@
       </inertial> -->
     </link>
-    <gazebo reference="laser_frame">
+<gazebo reference="laser_frame">
         <mu1 value="400"/>
         <mu2 value="400"/>
