Commit message: ros2_control

File: 3.0.0/src/scootbot/description/model.xacro (robot description, xacro)
@@ -13,5 +13,5 @@
   <xacro:property name="wheel_zoff" value="0.01"/>
   <xacro:property name="wheel_xoff" value="0.20"/>
-  <xacro:property name="caster_radius" value="0.071"/>
+  <!-- <xacro:property name="caster_radius" value="0.08"/> -->
   <xacro:property name="caster_width" value="0.047"/>
   <xacro:property name="caster_ygap" value="-0.285"/>
@@ -88,5 +88,5 @@
         <origin xyz="${col_x} ${col_y} ${col_z}" rpy="${pi/2} 0 ${mirror} "/>
         <geometry>
-            <cylinder radius="0.14" length="0.09"/>
+            <cylinder radius="0.13" length="0.09"/>
         </geometry>
         <material name="Gray">
@@ -115,5 +115,5 @@
     <link name="caster_frame_${prefix}_link">
       <visual>
-        <origin xyz="0.22 -0.005 0.075" rpy="0 0 0"/>
+        <origin xyz="0.22 -0.005 0.074" rpy="0 0 0"/>
         <geometry>
             <mesh filename="file:///$(find scootbot)/description/models/caster_frame.obj" scale="0.001 0.001 0.001"/>
@@ -140,7 +140,7 @@
     </joint>
     <gazebo reference="caster_frame_${prefix}_link">
-      <mu1 value="1.0"/>
-			<mu2 value="1.0"/>
-			<kp value="10000000.0" />
+      <mu1 value="0.7"/>
+			<mu2 value="0.9"/>
+			<kp value="2.0" />
 			<kd value="1.0" />
 			<fdir1 value="1 0 0"/>
@@ -150,9 +150,15 @@
 <xacro:caster_frame prefix="r" x_reflect="1" y_reflect="0.1752"/>
 <!-- Caster Wheels -->
-  <xacro:macro name="caster_wheel" params="prefix x_reflect y_reflect">
+  <xacro:macro name="caster_wheel" params="prefix x_reflect y_reflect caster_radius">
     <link name="casterwhl_${prefix}_link">
       <visual>
+              <contact>
+      <lateral_friction value="1.0"/>
+      <rolling_friction value="1.0"/>
+      <stiffness value="30000"/>
+      <damping value="1000"/>
+    </contact>
         <!-- <origin xyz="0.22 -0.165 -0.01" rpy="${pi/2} 0 0"/> -->
-        <origin xyz="0 0 0" rpy="${pi/2} 0 0"/>
+        <origin xyz="0 0 0.0" rpy="${pi/2} 0 0"/>
         <geometry>
             <cylinder radius="${caster_radius}" length="${caster_width}"/>
@@ -165,5 +171,5 @@
         <origin xyz="0 0 0" rpy="${pi/2} 0 0"/>
         <geometry>
-          <cylinder radius="0.075" length="0.05"/>
+          <cylinder radius="${caster_radius}" length="0.05"/>
           <!-- <sphere radius="0.1"/> -->
         </geometry>
@@ -180,6 +186,6 @@
     </joint>
     <gazebo reference="casterwhl_${prefix}_link">
-      <mu1 value="1.0"/>
-			<mu2 value="1.0"/>
+      <mu1 value="2000.0"/>
+			<mu2 value="1000.0"/>
 			<kp value="10000000.0" />
 			<kd value="1.0" />
@@ -187,6 +193,6 @@
     </gazebo>
   </xacro:macro>
-  <xacro:caster_wheel prefix="l" x_reflect="1" y_reflect="0.47"/>
-  <xacro:caster_wheel prefix="r" x_reflect="1" y_reflect="-0.47"/>
+  <xacro:caster_wheel prefix="l" x_reflect="1" y_reflect="0.47" caster_radius="0.0721"/>
+  <xacro:caster_wheel prefix="r" x_reflect="1" y_reflect="-0.47" caster_radius="0.072"/>
  <joint name="laser_joint" type="fixed">
         <parent link="base_link"/>

Commit message: controll tweaking

File: 3.0.0/src/scootbot/description/model.xacro (robot description, xacro)
@@ -219,4 +219,17 @@
       </inertial> -->
     </link>
+<!-- <joint name="imu_joint" type="fixed">
+        <parent link="base_link"/>
+        <child link="imu_link"/>
+        <origin xyz="0.45 -0.005 0.18" rpy="0 0 0"/>
+    </joint>
+        <link name="imu_link">
+      <visual>
+        <origin xyz="0 0 0" rpy="0 0 0"/>
+        <geometry>
+            <cylinder radius="0.02" length="0.02"/>
+        </geometry>
+      </visual>
+    </link>  -->
 <gazebo reference="laser_frame">
         <mu1 value="400"/>

File: 3.0.0/src/scootbot/description/ros2_control.xacro (robot description, xacro)
@@ -7,5 +7,5 @@
             <param name="right_wheel_name">drivewhl_r_joint</param>
             <param name="loop_rate">30</param>
-            <param name="device">/dev/ttyUSB0</param>
+            <param name="device">/dev/saber_serial</param>
             <param name="baud_rate">115200</param>
             <param name="timeout">1000</param>

Commit message: tweaks

File: 3.0.0/src/scootbot/description/model.xacro (robot description, xacro)
@@ -198,5 +198,5 @@
         <parent link="base_link"/>
         <child link="laser_frame"/>
-        <origin xyz="0.25 -0.005 0.18" rpy="0 0 0"/>
+        <origin xyz="0.25 -0.005 0.18" rpy="0 0 3.14159"/>
     </joint>
         <link name="laser_frame">
